File: Power Selector Board/PCB_Droit.kicad_sch (KiCad schematic)
At the start: 23 parts, among them J101 MSD-DB01M-12P, J102 MSD-DB01F-12P_1, J103 64900221122, J104 64900221122, J105 64900221122, J106 1998865, K101 G6SK-2G DC24, K102 J115F11C24VDCSH.9, K103 J115F11C24VDCSH.9, U102 LMW78_24-0.3RL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

Commit message: Premier commit pour routing PCB. Modif footprint connecteur batterie.
Parts:
- added H1, H2, H3, H4: Mounting-Hole-M3, Connectors:Mounting_Hole_3mm, symbol Mechanicals:Mounting-Hole-M3
- F101, F102: Current Rating (A) 30A -> 6.3A
- J101, J102: footprint Connectors:649012227222 -> Connectors:MSD-DB01F-12P-V2.0
Changed lines of the file:
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@@
       (effects (font (size 1.524 1.524)) hide)
     )
-    (property "Current Rating (A)" "30A" (at 77.47 104.14 0)
+    (property "Current Rating (A)" "6.3A" (at 77.47 104.14 0)
       (effects (font (size 1.27 1.27)))
     )
@@
     )
   )
+  (symbol (lib_id "Mechanicals:Mounting-Hole-M3") (at 48.26 195.58 0) (unit 1)
+    (in_bom yes) (on_board yes) (dnp no) (fields_autoplaced)
+    (property "Reference" "H2" (at 53.34 194.31 0)
+      (effects (font (size 1.524 1.524)) (justify left))
+    )
+    (property "Value" "Mounting-Hole-M3" (at 53.34 196.85 0)
+      (effects (font (size 1.524 1.524)) (justify left))
+    )
+    (property "Footprint" "Connectors:Mounting_Hole_3mm" (at 48.26 209.55 0)
+      (effects (font (size 1.524 1.524)) hide)
+    )
+    (property "Datasheet" "" (at 48.26 200.66 0)
+      (effects (font (size 1.524 1.524)) hide)
+    )
+    (pin "1")
+    (instances
+      (project "Power Selector"
+        (path "/809bdac1-fe7e-479d-b3c2-abd6ebce72b5/01a8522b-18e6-465b-b2cb-1d0f4aea8e80"
+          (reference "H2") (unit 1)
+        )
+      )
+    )
+  )
   (symbol (lib_id "Power_Port:GND_D") (at 170.18 228.6 0) (unit 1)
     (in_bom yes) (on_board yes) (dnp no)
@@
       (effects (font (size 1.524 1.524)))
     )
-    (property "Footprint" "Connectors:649012227222" (at 60.96 156.21 0)
+    (property "Footprint" "Connectors:MSD-DB01F-12P-V2.0" (at 60.96 156.21 0)
       (effects (font (size 1.524 1.524)) hide)
     )
@@
     )
   )
+  (symbol (lib_id "Mechanicals:Mounting-Hole-M3") (at 48.26 208.28 0) (unit 1)
+    (in_bom yes) (on_board yes) (dnp no) (fields_autoplaced)
+    (property "Reference" "H3" (at 53.34 207.01 0)
+      (effects (font (size 1.524 1.524)) (justify left))
+    )
+    (property "Value" "Mounting-Hole-M3" (at 53.34 209.55 0)
+      (effects (font (size 1.524 1.524)) (justify left))
+    )
+    (property "Footprint" "Connectors:Mounting_Hole_3mm" (at 48.26 222.25 0)
+      (effects (font (size 1.524 1.524)) hide)
+    )
+    (property "Datasheet" "" (at 48.26 213.36 0)
+      (effects (font (size 1.524 1.524)) hide)
+    )
+    (pin "1")
+    (instances
+      (project "Power Selector"
+        (path "/809bdac1-fe7e-479d-b3c2-abd6ebce72b5/01a8522b-18e6-465b-b2cb-1d0f4aea8e80"
+          (reference "H3") (unit 1)
+        )
+      )
+    )
+  )
   (symbol (lib_id "Power_Port:GND_D") (at 334.01 123.19 0) (unit 1)
     (in_bom yes) (on_board yes) (dnp no)
@@
       (effects (font (size 1.524 1.524)) hide)
     )
-    (property "Current Rating (A)" "30A" (at 74.93 74.93 0)
+    (property "Current Rating (A)" "6.3A" (at 74.93 74.93 0)
       (effects (font (size 1.27 1.27)))
     )
@@
         (path "/809bdac1-fe7e-479d-b3c2-abd6ebce72b5/01a8522b-18e6-465b-b2cb-1d0f4aea8e80"
           (reference "#PWR0329") (unit 1)
+        )
+      )
+    )
+  )
+  (symbol (lib_id "Mechanicals:Mounting-Hole-M3") (at 48.26 222.25 0) (unit 1)
+    (in_bom yes) (on_board yes) (dnp no) (fields_autoplaced)
+    (property "Reference" "H4" (at 53.34 220.98 0)
+      (effects (font (size 1.524 1.524)) (justify left))
+    )
+    (property "Value" "Mounting-Hole-M3" (at 53.34 223.52 0)
+      (effects (font (size 1.524 1.524)) (justify left))
+    )
+    (property "Footprint" "Connectors:Mounting_Hole_3mm" (at 48.26 236.22 0)
+      (effects (font (size 1.524 1.524)) hide)
+    )
+    (property "Datasheet" "" (at 48.26 227.33 0)
+      (effects (font (size 1.524 1.524)) hide)
+    )
+    (pin "1")
+    (instances
+      (project "Power Selector"
+        (path "/809bdac1-fe7e-479d-b3c2-abd6ebce72b5/01a8522b-18e6-465b-b2cb-1d0f4aea8e80"
+          (reference "H4") (unit 1)
         )
       )
@@
     )
   )
+  (symbol (lib_id "Mechanicals:Mounting-Hole-M3") (at 48.26 182.88 0) (unit 1)
+    (in_bom yes) (on_board yes) (dnp no) (fields_autoplaced)
+    (property "Reference" "H1" (at 53.34 181.61 0)
+      (effects (font (size 1.524 1.524)) (justify left))
+    )
+    (property "Value" "Mounting-Hole-M3" (at 53.34 184.15 0)
+      (effects (font (size 1.524 1.524)) (justify left))
+    )
+    (property "Footprint" "Connectors:Mounting_Hole_3mm" (at 48.26 196.85 0)
+      (effects (font (size 1.524 1.524)) hide)
+    )
+    (property "Datasheet" "" (at 48.26 187.96 0)
+      (effects (font (size 1.524 1.524)) hide)
+    )
+    (pin "1")
+    (instances
+      (project "Power Selector"
+        (path "/809bdac1-fe7e-479d-b3c2-abd6ebce72b5/01a8522b-18e6-465b-b2cb-1d0f4aea8e80"
+          (reference "H1") (unit 1)
+        )
+      )
+    )
+  )
   (symbol (lib_id "Fuses:0698Q2000-02") (at 226.06 214.63 0) (unit 1)
     (in_bom yes) (on_board yes) (dnp no) (fields_autoplaced)
@@
       (effects (font (size 1.524 1.524)))
     )
-    (property "Footprint" "Connectors:649012227222" (at 342.9 148.59 0)
-      (effects (font (size 1.524 1.524)) hide)
-    )
+    (property "Footprint" "Connectors:MSD-DB01F-12P-V2.0" (at 342.9 148.59 0)
+      (effects (font (size 1.524 1.524)) hide)
+    )
